Commit message: underwater

File: definition/robots/eca_a9_default.urdf.xacro (robot description, xacro)
@@ -17,5 +17,5 @@
   <xacro:arg name="inertial_reference_frame" default="world"/>
   <!-- Include the UUV macro file -->
-  <xacro:include filename="$(find configuration)/urdf/eca_a9_base.xacro"/>
+  <xacro:include filename="$(find definition)/urdf/eca_a9_base.xacro"/>
   <!-- Create the eca_a9 -->
   <xacro:eca_a9_base

File: definition/urdf/eca_a9_base.xacro (robot description, xacro)
@@ -28,8 +28,8 @@
   <xacro:property name="area" value="0.04155"/>
   <xacro:property name="length" value="1.98"/>
-  <xacro:property name="visual_mesh_file" value="file://$(find configuration)/mesh/eca_a9.dae"/>
-  <xacro:property name="collision_mesh_file" value="file://$(find configuration)/mesh/eca_a9.stl"/>
-  <xacro:property name="prop_mesh_file" value="file://$(find configuration)/mesh/eca_a9_propeller.dae"/>
-  <xacro:property name="fin_mesh_file" value="file://$(find configuration)/mesh/eca_a9_fin.dae"/>
+  <xacro:property name="visual_mesh_file" value="file://$(find definition)/mesh/eca_a9.dae"/>
+  <xacro:property name="collision_mesh_file" value="file://$(find definition)/mesh/eca_a9.stl"/>
+  <xacro:property name="prop_mesh_file" value="file://$(find definition)/mesh/eca_a9_propeller.dae"/>
+  <xacro:property name="fin_mesh_file" value="file://$(find definition)/mesh/eca_a9_fin.dae"/>
   <xacro:macro name="eca_a9_base" params="namespace debug inertial_reference_frame">
     <link name="${namespace}/base_link">
